Commit message: “constraint_planning”

File: mujoco_models/bimanual.urdf (robot description, URDF)
Before this commit: robot bimanual, 38 links, 37 joints
Links:
- removed link pot_link
Joints:
- removed joint pot_free_joint

Commit message: path_simplification

File: mujoco_models/bimanual.urdf (robot description, URDF)
Before this commit: robot bimanual, 37 links, 36 joints
Links:
- added link pot_link, mass 5.35e-1; collision box size=0.01 0.16 0.10; collision box size=0.01 0.16 0.10
- link arm_base_link: geometry collision mesh filename=package://new_bimanual_pkg/mujoco_models/assets/ffw_bg2/bod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 scale=0.001 0.001 0.001; visual mesh filename=package://new_bimanual_pkg/mujoco_models/assets/ffw_bg2/bod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 scale=0.001 0.001 0.001
- link arm_l_link1: geometry collision mesh filename=package://new_bimanual_pkg/mujoco_models/assets/ffw_bg2/arm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 scale=0.001 0.001 0.001; visual mesh filename=package://new_bimanual_pkg/mujoco_models/assets/ffw_bg2/arm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 scale=0.001 0.001 0.001
- link arm_l_link2: geometry collision mesh filename=package://new_bimanual_pkg/mujoco_models/assets/ffw_bg2/arm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 scale=0.001 0.001 0.001; visual mesh filename=package://new_bimanual_pkg/mujoco_models/assets/ffw_bg2/arm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 scale=0.001 0.001 0.001
- link arm_l_link3: geometry collision mesh filename=package://new_bimanual_pkg/mujoco_models/assets/ffw_bg2/arm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 scale=0.001 0.001 0.001; visual mesh filename=package://new_bimanual_pkg/mujoco_models/assets/ffw_bg2/arm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 scale=0.001 0.001 0.001
- link arm_l_link4: geometry collision mesh filename=package://new_bimanual_pkg/mujoco_models/assets/ffw_bg2/arm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 scale=0.001 0.001 0.001; visual mesh filename=package://new_bimanual_pkg/mujoco_models/assets/ffw_bg2/arm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 scale=0.001 0.001 0.001
- link arm_l_link5: geometry collision mesh filename=package://new_bimanual_pkg/mujoco_models/assets/ffw_bg2/arm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 scale=0.001 0.001 0.001; visual mesh filename=package://new_bimanual_pkg/mujoco_models/assets/ffw_bg2/arm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 scale=0.001 0.001 0.001
- link arm_l_link6: geometry collision mesh filename=package://new_bimanual_pkg/mujoco_models/assets/ffw_bg2/arm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 scale=0.001 0.001 0.001; visual mesh filename=package://new_bimanual_pkg/mujoco_models/assets/ffw_bg2/arm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 scale=0.001 0.001 0.001
- link arm_l_link7: geometry collision mesh filename=package://new_bimanual_pkg/mujoco_models/assets/ffw_bg2/arm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 scale=0.001 0.001 0.001; visual mesh filename=package://new_bimanual_pkg/mujoco_models/assets/ffw_bg2/arm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 scale=0.001 0.001 0.001
- link arm_r_link1: geometry collision mesh filename=package://new_bimanual_pkg/mujoco_models/assets/ffw_bg2/arm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 scale=0.001 0.001 0.001; visual mesh filename=package://new_bimanual_pkg/mujoco_models/assets/ffw_bg2/arm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 scale=0.001 0.001 0.001
- link arm_r_link2: geometry collision mesh filename=package://new_bimanual_pkg/mujoco_models/assets/ffw_bg2/arm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 scale=0.001 0.001 0.001; visual mesh filename=package://new_bimanual_pkg/mujoco_models/assets/ffw_bg2/arm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 scale=0.001 0.001 0.001
- link arm_r_link3: geometry collision mesh filename=package://new_bimanual_pkg/mujoco_models/assets/ffw_bg2/arm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 scale=0.001 0.001 0.001; visual mesh filename=package://new_bimanual_pkg/mujoco_models/assets/ffw_bg2/arm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 scale=0.001 0.001 0.001
- link arm_r_link4: geometry collision mesh filename=package://new_bimanual_pkg/mujoco_models/assets/ffw_bg2/arm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 scale=0.001 0.001 0.001; visual mesh filename=package://new_bimanual_pkg/mujoco_models/assets/ffw_bg2/arm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 scale=0.001 0.001 0.001
- link arm_r_link5: geometry collision mesh filename=package://new_bimanual_pkg/mujoco_models/assets/ffw_bg2/arm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 scale=0.001 0.001 0.001; visual mesh filename=package://new_bimanual_pkg/mujoco_models/assets/ffw_bg2/arm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 scale=0.001 0.001 0.001
- link arm_r_link6: geometry collision mesh filename=package://new_bimanual_pkg/mujoco_models/assets/ffw_bg2/arm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 scale=0.001 0.001 0.001; visual mesh filename=package://new_bimanual_pkg/mujoco_models/assets/ffw_bg2/arm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 scale=0.001 0.001 0.001
- link arm_r_link7: geometry collision mesh filename=package://new_bimanual_pkg/mujoco_models/assets/ffw_bg2/arm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 scale=0.001 0.001 0.001; visual mesh filename=package://new_bimanual_pkg/mujoco_models/assets/ffw_bg2/arm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 scale=0.001 0.001 0.001
- link base_link: geometry collision mesh filename=package://new_bimanual_pkg/mujoco_models/assets/ffw_bg2/bas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 scale=0.001 0.001 0.001; visual mesh filename=package://new_bimanual_pkg/mujoco_models/assets/ffw_bg2/bas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 scale=0.001 0.001 0.001
- link gripper_l_rh_p12_rn_base: geometry collision mesh filename=package://new_bimanual_pkg/mujoco_models/assets/ffw_bg2/bas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 scale=0.001 0.001 0.001; visual mesh filename=package://new_bimanual_pkg/mujoco_models/assets/ffw_bg2/bas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 scale=0.001 0.001 0.001
- link gripper_l_rh_p12_rn_l1: geometry collision mesh filename=package://new_bimanual_pkg/mujoco_models/assets/ffw_bg2/l1.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 scale=0.001 0.001 0.001; visual mesh filename=package://new_bimanual_pkg/mujoco_models/assets/ffw_bg2/l1.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 scale=0.001 0.001 0.001
- link gripper_l_rh_p12_rn_l2: geometry collision mesh filename=package://new_bimanual_pkg/mujoco_models/assets/ffw_bg2/l2.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 scale=0.001 0.001 0.001; visual mesh filename=package://new_bimanual_pkg/mujoco_models/assets/ffw_bg2/l2.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 scale=0.001 0.001 0.001
- link gripper_l_rh_p12_rn_r1: geometry collision mesh filename=package://new_bimanual_pkg/mujoco_models/assets/ffw_bg2/r1.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 scale=0.001 0.001 0.001; visual mesh filename=package://new_bimanual_pkg/mujoco_models/assets/ffw_bg2/r1.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 scale=0.001 0.001 0.001
- link gripper_l_rh_p12_rn_r2: geometry collision mesh filename=package://new_bimanual_pkg/mujoco_models/assets/ffw_bg2/r2.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 scale=0.001 0.001 0.001; visual mesh filename=package://new_bimanual_pkg/mujoco_models/assets/ffw_bg2/r2.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 scale=0.001 0.001 0.001
- link gripper_r_rh_p12_rn_base: geometry collision mesh filename=package://new_bimanual_pkg/mujoco_models/assets/ffw_bg2/bas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 scale=0.001 0.001 0.001; visual mesh filename=package://new_bimanual_pkg/mujoco_models/assets/ffw_bg2/bas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 scale=0.001 0.001 0.001
- link gripper_r_rh_p12_rn_l1: geometry collision mesh filename=package://new_bimanual_pkg/mujoco_models/assets/ffw_bg2/l1.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 scale=0.001 0.001 0.001; visual mesh filename=package://new_bimanual_pkg/mujoco_models/assets/ffw_bg2/l1.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 scale=0.001 0.001 0.001
- link gripper_r_rh_p12_rn_l2: geometry collision mesh filename=package://new_bimanual_pkg/mujoco_models/assets/ffw_bg2/l2.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 scale=0.001 0.001 0.001; visual mesh filename=package://new_bimanual_pkg/mujoco_models/assets/ffw_bg2/l2.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 scale=0.001 0.001 0.001
- link gripper_r_rh_p12_rn_r1: geometry collision mesh filename=package://new_bimanual_pkg/mujoco_models/assets/ffw_bg2/r1.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 scale=0.001 0.001 0.001; visual mesh filename=package://new_bimanual_pkg/mujoco_models/assets/ffw_bg2/r1.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 scale=0.001 0.001 0.001
- link gripper_r_rh_p12_rn_r2: geometry collision mesh filename=package://new_bimanual_pkg/mujoco_models/assets/ffw_bg2/r2.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 scale=0.001 0.001 0.001; visual mesh filename=package://new_bimanual_pkg/mujoco_models/assets/ffw_bg2/r2.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 scale=0.001 0.001 0.001
- link head_link1: geometry collision mesh filename=package://new_bimanual_pkg/mujoco_models/assets/ffw_bg2/hea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 scale=0.001 0.001 0.001; visual mesh filename=package://new_bimanual_pkg/mujoco_models/assets/ffw_bg2/hea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 scale=0.001 0.001 0.001
- link head_link2: geometry collision mesh filename=package://new_bimanual_pkg/mujoco_models/assets/ffw_bg2/hea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 scale=0.001 0.001 0.001; visual mesh filename=package://new_bimanual_pkg/mujoco_models/assets/ffw_bg2/hea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 scale=0.001 0.001 0.001
- link left_wheel_drive_link: geometry collision mesh filename=package://new_bimanual_pkg/mujoco_models/assets/ffw_bg2/lef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 scale=0.001 0.001 0.001; visual mesh filename=package://new_bimanual_pkg/mujoco_models/assets/ffw_bg2/lef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 scale=0.001 0.001 0.001
- link left_wheel_steer_link: geometry collision mesh filename=package://new_bimanual_pkg/mujoco_models/assets/ffw_bg2/lef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 scale=0.001 0.001 0.001; visual mesh filename=package://new_bimanual_pkg/mujoco_models/assets/ffw_bg2/lef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 scale=0.001 0.001 0.001
- link lift_link: geometry collision mesh filename=package://new_bimanual_pkg/mujoco_models/assets/ffw_bg2/lif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 scale=0.001 0.001 0.001; visual mesh filename=package://new_bimanual_pkg/mujoco_models/assets/ffw_bg2/lif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 scale=0.001 0.001 0.001
- link rear_wheel_drive_link: geometry collision mesh filename=package://new_bimanual_pkg/mujoco_models/assets/ffw_bg2/rea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 scale=0.001 0.001 0.001; visual mesh filename=package://new_bimanual_pkg/mujoco_models/assets/ffw_bg2/rea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 scale=0.001 0.001 0.001
- link rear_wheel_steer_link: geometry collision mesh filename=package://new_bimanual_pkg/mujoco_models/assets/ffw_bg2/rea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 scale=0.001 0.001 0.001; visual mesh filename=package://new_bimanual_pkg/mujoco_models/assets/ffw_bg2/rea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 scale=0.001 0.001 0.001
- link right_wheel_drive_link: geometry collision mesh filename=package://new_bimanual_pkg/mujoco_models/assets/ffw_bg2/rig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 scale=0.001 0.001 0.001; visual mesh filename=package://new_bimanual_pkg/mujoco_models/assets/ffw_bg2/rig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 scale=0.001 0.001 0.001
- link right_wheel_steer_link: geometry collision mesh filename=package://new_bimanual_pkg/mujoco_models/assets/ffw_bg2/rig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 scale=0.001 0.001 0.001; visual mesh filename=package://new_bimanual_pkg/mujoco_models/assets/ffw_bg2/rig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 scale=0.001 0.001 0.001
- link table_link: geometry collision box size=0.07 0.07 1.0; collision box size=0.07 0.07 1.0
Joints:
- added joint pot_free_joint: type floating, parent world, child pot_link, origin xyz=0.5 0.0 1.01 rpy=0 0 0

Commit message: all modified

File: mujoco_models/bimanual.urdf (robot description, URDF)
Before this commit: robot bimanual, 38 links, 37 joints
Links:
- removed link pot_link
- removed link table_link
- added link kitchen_sink; collision box size=0.15 0.15 0.03; collision box size=0.4 0.95 1.05
Joints:
- removed joint pot_free_joint
- removed joint table_fixed_joint
- added joint kitchen_sink_fixed: type fixed, parent world, child kitchen_sink, origin xyz=0.87 0.48 -0.033 rpy=0 0 0
